File: board/TinyTony_ShenzenReady.sch (EAGLE design)
At the start: 7 parts, among them U1 ATTINY85

Commit message: board
Parts:
- ISP1: value AVRISP-6 -> AVRISPPOGO; device adafruit:AVRISP-6 -> tinytony_shenzenReady:AVRISPPOGO
Changed lines of the file:
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@@
 <part name="GND2" library="tinytony_shenzenReady" deviceset="GND" device=""/>
 <part name="SUPPLY2" library="SparkFun-PowerSymbols" deviceset="VCC" device=""/>
-<part name="ISP1" library="adafruit" deviceset="AVRISP" device="-6"/>
+<part name="ISP1" library="tinytony_shenzenReady" deviceset="AVRISP" device="POGO"/>
 <part name="GND3" library="tinytony_shenzenReady" deviceset="GND" device=""/>
 <part name="SUPPLY3" library="SparkFun-PowerSymbols" deviceset="VCC" device=""/>

Commit message: 2 drivers and cap
Parts:
- added C1, C2: (no value), microbuilder:CAP_CERAMIC0805-NOTHERMALS
- added JP3: MOTOR2, tinytony_shenzenReady:HEADER-1X2ROUND
- added U$2, U$3: DRV8830, tinytony_shenzenReady:DRV8830
- JP2: value motor driver -> MOTOR1
Connections:
- new net N$1: U$3.A1
- new net N$2: JP3.1, U$3.OUT1
- new net N$3: JP2.1, U$2.OUT1
- new net N$4: JP2.2, U$2.OUT2
- new net N$5: JP3.2, U$3.OUT2
- new net N$8: U$2.A0
- net 5: now also U$2.SCL, U$3.SCL; no longer JP2.1
- net 7: now also U$2.SDA, U$3.SDA
- net GND: now also C1.P$1, C2.P$1, U$2.A1, U$2.GND, U$3.A0, U$3.GND
- net VCC: now also C1.P$2, C2.P$2, U$2.VCC, U$3.VCC; no longer JP2.2
Other:
- note added: "ANALOG_IN"
- note added: "IR_RECIVE"
- note added: "SCL"
- note added: "SDA"
- note added: "SERIAL"
- note added: "addr: 0xC3h"
- note added: "addr: 0xC7h"
- moved on the sheet: ISP1, JP1, R1, R2, U$1, U1

Commit message: bigger, 1206cp
Parts:
- removed R1, R2: PHOTOCELLPTH, SparkFun-Sensors:PHOTOCELLPTH
- added PHOTOCELL01, PHOTOCELL02: PHOTOCELL0N1, TinyTony_ShenzenReady:PHOTOCELL0N1
- C1, C2: device microbuilder:CAP_CERAMIC0805-NOTHERMALS -> TinyTony_ShenzenReady:CAP_CERAMIC1206
Connections:
- net 2: now also PHOTOCELL01.1, PHOTOCELL02.2; no longer R1.P$2, R2.P$1
- net GND: now also PHOTOCELL01.2; no longer R1.P$1
- net VCC: now also PHOTOCELL02.1; no longer R2.P$2
